File: kicad/remote/lux/lux.kicad_sch (KiCad schematic)
At the start: 24 parts, among them T1 trace, U1 ESP32-S3-WROOM-1U-N16R8, U2 TPS63020DSJR

Commit message: i
Parts:
- added SW1, SW2, SW3, SW4: sw, Button_Switch_THT:SW_PUSH_6mm_H5mm, symbol Switch:SW_Push
Connections:
- net GND: now also SW1.2, SW2.2, SW3.2, SW4.2
- net IO4: now also SW1.1
- net IO5: now also SW2.1
- net IO6: now also SW3.1
- net IO7: now also SW4.1
- net IO10: no longer names the net of U1.18 (IO10)
- net IO11: no longer names the net of U1.19 (IO11)
- net IO35: no longer names the net of U1.29 (IO36)
- net IO36: no longer names the net of U1.28 (IO35)
- net IO41: no longer names the net of U1.34 (IO41)
- net IO42: no longer names the net of U1.35 (IO42)
- no-connect marks 29 -> 33
