File: kicad/remote/remote.kicad_pcb (KiCad board)
At the start: 4 copper layers, 73.5 x 45.5 mm, 28 parts, among them SW1 sw, SW2 sw, SW3 sw, SW4 sw, T1 trace, U1 ESP32-S3-WROOM-1U-N16R8, U2 TPS63020DSJR

Commit message: sept 17
Parts:
- removed SW3, SW4: sw, Button_Switch_THT:SW_PUSH_6mm_H5mm
- added D1: Yellow, LED_SMD:LED_1206_3216Metric, F.Cu at (870.5, 619.0)
- added D2: WHITE, LED_SMD:LED_1206_3216Metric, F.Cu at (868.4, 609.5)
- added D3: Yellow, LED_SMD:LED_1206_3216Metric, F.Cu at (883.5, 636.5)
- added J1: joystick, Connector_PinHeader_2.54mm:PinHeader_1x05_P2.54mm_Vertical, F.Cu at (850.0, 606.6)
- added J2: joystick, Connector_PinHeader_2.54mm:PinHeader_1x05_P2.54mm_Vertical, F.Cu at (919.5, 606.6)
- added R10: 220 ohm, Resistor_SMD:R_0603_1608Metric, F.Cu at (880.0, 633.0)
- added R11: 220 ohm, Resistor_SMD:R_0603_1608Metric, F.Cu at (884.7, 633.0)
- added R8: 220 ohm, Resistor_SMD:R_0603_1608Metric, F.Cu at (874.0, 617.0)
- added R9: 220 ohm, Resistor_SMD:R_0603_1608Metric, F.Cu at (871.8, 613.5)
- moved SW2 20.5 mm to (859.5, 628.5)
- moved SW1 19.5 mm to (859.0, 617.5)
- moved BT1 10.0 mm to (883.0, 596.0)
- moved C20 10.0 mm to (908.5, 597.0)
- moved C21 10.0 mm to (903.5, 597.0)
- moved C22 10.0 mm to (894.0, 597.0)
- moved C23 10.0 mm to (889.5, 597.0)
Connections:
- SW1 pad 1: /IO4 -> /IO15
- SW2 pad 1: /IO5 -> /IO16
- U1 pad 10: unconnected-(U1-IO17-Pad10) -> /IO17
- U1 pad 11: unconnected-(U1-IO18-Pad11) -> /IO18
- U1 pad 4: /IO4 -> /J1x
- U1 pad 5: /IO5 -> /J1y
- U1 pad 6: /IO6 -> /J2x
- U1 pad 7: /IO7 -> /J2y
- U1 pad 8: unconnected-(U1-IO15-Pad8) -> /IO15
- U1 pad 9: unconnected-(U1-IO16-Pad9) -> /IO16
Routing:
- net +3.3V: track 81.5 -> 154.8 mm, vias 8 -> 10
- net /J2y: track 0.00 -> 49.4 mm, vias 0 -> 1
- net /J2x: track 0.00 -> 44.8 mm, vias 0 -> 1
- net /J1y: track 0.00 -> 36.8 mm, vias 0 -> 1
- net /J1x: track 0.00 -> 32.3 mm, vias 0 -> 1
- net /IO7: track 27.9 -> 0.00 mm, vias 1 -> 0
- net /IO16: track 0.00 -> 27.1 mm
- net /IO4: track 26.0 -> 0.00 mm, vias 1 -> 0
- net /IO6: track 22.3 -> 0.00 mm, vias 1 -> 0
- net /IO5: track 22.2 -> 0.00 mm, vias 1 -> 0
- net +5V: track 41.1 -> 62.8 mm, vias 4 -> 5
- net /IO15: track 0.00 -> 21.2 mm
- net /IO18: track 0.00 -> 10.3 mm, vias 0 -> 2
- net Net-(R10-Pad1): track 0.00 -> 8.40 mm
- net Net-(D2-K): track 0.00 -> 5.66 mm
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
Commit message: sep 18
Parts:
- added H3: MountingHole, MountingHole:MountingHole_2.5mm, F.Cu at (844.0, 635.0)
- added H4: MountingHole, MountingHole:MountingHole_2.5mm, F.Cu at (927.5, 634.5)
- added H5: MountingHole, MountingHole:MountingHole_2.5mm, F.Cu at (871.5, 597.5)
- moved J2 10.2 mm to (919.5, 596.4), turned to 0 degrees
- moved H1 6.40 mm to (846.5, 613.0)
- moved H2 6.40 mm to (923.0, 611.5)
Connections:
- J1 pad 5: unconnected-(J1-Pin_5-Pad5) -> /IO12
- J2 pad 5: unconnected-(J2-Pin_5-Pad5) -> /IO13
- U1 pad 20: unconnected-(U1-IO12-Pad20) -> /IO12
- U1 pad 21: unconnected-(U1-IO13-Pad21) -> /IO13
Routing:
- net /IO12: track 0.00 -> 51.4 mm, vias 0 -> 1
- net /IO13: track 0.00 -> 38.8 mm, vias 0 -> 1
- net /J2y: track 49.4 -> 55.1 mm
- net Net-(T1-Pin_1): track 15.9 -> 21.3 mm
- net +3.3V: track 154.8 -> 160.0 mm
Other:
- board size 73.5 x 45.5 mm -> 90 x 45 mm

Commit message: sept 19
Parts:
- moved H1 1.00 mm to (846.5, 612.0)
Changed lines of the file:
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@@
 		(model "/home/erox/Downloads/joy_stick_a2/joy_stick_2a.step"
 			(offset
-				(xyz -1.5 -17 0)
+				(xyz -2 -18.2 0)
 			)
 			(scale
@@
 	(footprint "MountingHole:MountingHole_2.5mm"
 		(layer "F.Cu")
-		(at 846.5 613)
+		(at 846.5 612)
 		(descr "Mounting Hole 2.5mm, no annular, generated by kicad-footprint-generator mountinghole.py")
 		(tags "mountinghole")
@@
 		(model "/home/erox/Downloads/joy_stick_a2/joy_stick_2a.step"
 			(offset
-				(xyz -1.5 -18 0)
+				(xyz -2 -18.2 0)
 			)
 			(scale
@@
 	)
 	(segment
+		(start 887.115 623.370002)
+		(end 887.115 622.115)
+		(width 0.2)
+		(layer "F.Cu")
+		(net "/IO12")
+	)
+	(segment
+		(start 887.115 622.115)
+		(end 886 621)
+		(width 0.2)
+		(layer "F.Cu")
+		(net "/IO12")
+	)
+	(via
+		(at 886 621)
+		(size 0.6)
+		(drill 0.3)
+		(layers "F.Cu" "B.Cu")
+		(net "/IO12")
+	)
+	(segment
+		(start 858.18 604.6)
+		(end 850 596.42)
+		(width 0.2)
+		(layer "B.Cu")
+		(net "/IO12")
+	)
+	(segment
+		(start 878.15 613.15)
+		(end 878.15 609.023655)
+		(width 0.2)
+		(layer "B.Cu")
+		(net "/IO12")
+	)
+	(segment
+		(start 886 621)
+		(end 878.15 613.15)
+		(width 0.2)
+		(layer "B.Cu")
+		(net "/IO12")
+	)
+	(segment
+		(start 873.726345 604.6)
+		(end 858.18 604.6)
+		(width 0.2)
+		(layer "B.Cu")
+		(net "/IO12")
+	)
+	(segment
+		(start 878.15 609.023655)
+		(end 873.726345 604.6)
+		(width 0.2)
+		(layer "B.Cu")
+		(net "/IO12")
+	)
+	(segment
+		(start 888.385 622.115)
+		(end 893 617.5)
+		(width 0.2)
+		(layer "F.Cu")
+		(net "/IO13")
+	)
+	(segment
+		(start 888.385 623.370002)
+		(end 888.385 622.115)
+		(width 0.2)
+		(layer "F.Cu")
+		(net "/IO13")
+	)
+	(via
+		(at 893 617.5)
+		(size 0.6)
+		(drill 0.3)
+		(layers "F.Cu" "B.Cu")
+		(net "/IO13")
+	)
+	(segment
+		(start 893 617.5)
+		(end 903.96 606.54)
+		(width 0.2)
+		(layer "B.Cu")
+		(net "/IO13")
+	)
+	(segment
+		(start 903.96 606.54)
+		(end 919.5 606.54)
+		(width 0.2)
+		(layer "B.Cu")
+		(net "/IO13")
+	)
+	(segment
 		(start 899 620.175)
 		(end 897.055 622.12)
@@
 		(net "Net-(USBC1-CC2)")
 	)
-	(segment
-		(start 887.115 623.370002)
-		(end 887.115 622.115)
-		(width 0.2)
-		(layer "F.Cu")
-		(net "/IO12")
-	)
-	(segment
-		(start 887.115 622.115)
-		(end 886 621)
-		(width 0.2)
-		(layer "F.Cu")
-		(net "/IO12")
-	)
-	(via
-		(at 886 621)
-		(size 0.6)
-		(drill 0.3)
-		(layers "F.Cu" "B.Cu")
-		(net "/IO12")
-	)
-	(segment
-		(start 858.18 604.6)
-		(end 850 596.42)
-		(width 0.2)
-		(layer "B.Cu")
-		(net "/IO12")
-	)
-	(segment
-		(start 878.15 613.15)
-		(end 878.15 609.023655)
-		(width 0.2)
-		(layer "B.Cu")
-		(net "/IO12")
-	)
-	(segment
-		(start 886 621)
-		(end 878.15 613.15)
-		(width 0.2)
-		(layer "B.Cu")
-		(net "/IO12")
-	)
-	(segment
-		(start 873.726345 604.6)
-		(end 858.18 604.6)
-		(width 0.2)
-		(layer "B.Cu")
-		(net "/IO12")
-	)
-	(segment
-		(start 878.15 609.023655)
-		(end 873.726345 604.6)
-		(width 0.2)
-		(layer "B.Cu")
-		(net "/IO12")
-	)
-	(segment
-		(start 888.385 622.115)
-		(end 893 617.5)
-		(width 0.2)
-		(layer "F.Cu")
-		(net "/IO13")
-	)
-	(segment
-		(start 888.385 623.370002)
-		(end 888.385 622.115)
-		(width 0.2)
-		(layer "F.Cu")
-		(net "/IO13")
-	)
-	(via
-		(at 893 617.5)
-		(size 0.6)
-		(drill 0.3)
-		(layers "F.Cu" "B.Cu")
-		(net "/IO13")
-	)
-	(segment
-		(start 893 617.5)
-		(end 903.96 606.54)
-		(width 0.2)
-		(layer "B.Cu")
-		(net "/IO13")
-	)
-	(segment
-		(start 903.96 606.54)
-		(end 919.5 606.54)
-		(width 0.2)
-		(layer "B.Cu")
-		(net "/IO13")
-	)
 	(zone

Commit message: sept 22 lol
Routing:
- net +5V: track 62.8 -> 51.7 mm, vias 5 -> 4
Changed lines of the file:
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@@
+	)
+	(segment
+		(start 912.398529 626)
+		(end 915.848529 629.45)
+		(width 0.3)
+		(layer "F.Cu")
+		(net "+5V")
 	)
 	(segment
@@
 		(end 892.6 631.507544)
 		(width 0.4)
+		(layer "F.Cu")
+		(net "+5V")
+	)
+	(segment
+		(start 907.825 626)
+		(end 912.398529 626)
+		(width 0.3)
+		(layer "F.Cu")
+		(net "+5V")
+	)
+	(segment
+		(start 915.848529 629.45)
+		(end 917.05 629.45)
+		(width 0.3)
 		(layer "F.Cu")
 		(net "+5V")
@@
 	)
 	(segment
+		(start 907.325 625.5)
+		(end 907.825 626)
+		(width 0.3)
+		(layer "F.Cu")
+		(net "+5V")
+	)
+	(segment
 		(start 909.02 625)
 		(end 909.000001 625)
@@
 		(width 0.4)
 		(layer "F.Cu")
-		(net "+5V")
-	)
-	(via
-		(at 896.886196 630.113804)
-		(size 0.5)
-		(drill 0.3)
-		(layers "F.Cu" "B.Cu")
 		(net "+5V")
 	)
@@
 	)
 	(segment
-		(start 896.886196 630.113804)
-		(end 903.5 630.113804)
-		(width 0.4)
-		(layer "In1.Cu")
-		(net "+5V")
-	)
-	(segment
 		(start 888.55 634.05)
 		(end 899.563804 634.05)
 		(width 0.2)
-		(layer "In1.Cu")
-		(net "+5V")
-	)
-	(segment
-		(start 903.5 630.113804)
-		(end 912.886196 630.113804)
-		(width 0.4)
 		(layer "In1.Cu")
 		(net "+5V")
@@
 		(end 908.000001 626)
 		(width 0.3)
-		(layer "In1.Cu")
-		(net "+5V")
-	)
-	(segment
-		(start 912.886196 630.113804)
-		(end 913.5 629.5)
-		(width 0.4)
 		(layer "In1.Cu")
 		(net "+5V")
@@
 		(layer "In1.Cu")
 		(net "+5V")
-	)
-	(segment
-		(start 899.563804 634.05)
-		(end 903.5 630.113804)
-		(width 0.2)
-		(layer "In1.Cu")
-		(net "+5V")

Commit message: readme more
Connections:
- C14 pad 2: +5V -> +5VA
- C15 pad 1: +5V -> +5VA
- D3 pad 2: +3.3V -> GND1
- R1 pad 1: +3.3V -> GND1
- R2 pad 1: +3.3V -> GND1
- R3 pad 2: +5V -> +5VA
- R5 pad 2: +3.3V -> GND1
- U2 pad 1: +5V -> +5VA
- U2 pad 10: +5V -> +5VA
- U2 pad 11: +5V -> +5VA
- U2 pad 12: +5V -> +5VA
- USBC1 pad A1B12: +3.3V -> GND1
- USBC1 pad B1A12: +3.3V -> GND1
Routing:
- net +5VA: track 26.5 -> 80.3 mm, vias 0 -> 3
- net +3.3V: track 160.0 -> 106.6 mm, vias 10 -> 7
- net GND1: track 0.00 -> 40.3 mm, vias 0 -> 3
- net +5V: track 51.7 -> 28.5 mm, vias 4 -> 2
- net GND: track 42.7 -> 45.3 mm, vias 13 -> 15
- net Net-(R10-Pad1): track 8.40 -> 7.77 mm
