File: kicad/remote/remote.kicad_sch (KiCad schematic)
At the start: 28 parts, among them SW1 sw, SW2 sw, SW3 sw, SW4 sw, T1 trace, U1 ESP32-S3-WROOM-1U-N16R8, U2 TPS63020DSJR

Commit message: sept 17
Parts:
- removed SW3, SW4: sw, Button_Switch_THT:SW_PUSH_6mm_H5mm, symbol Switch:SW_Push
- added D1, D3: Yellow, LED_SMD:LED_1206_3216Metric, symbol Device:LED
- added D2: WHITE, LED_SMD:LED_1206_3216Metric, symbol Device:LED
- added J1, J2: joystick, Connector_PinHeader_2.54mm:PinHeader_1x05_P2.54mm_Vertical, symbol Connector:Conn_01x05_Pin
- added R10, R11, R8, R9: 220 ohm, Resistor_SMD:R_0603_1608Metric, symbol Device:R
Connections:
- net +3.3V: now also D3.2 (A), J1.2 (Pin_2), J2.2 (Pin_2)
- net +5V: now also R11.1
- net GND: now also D1.2 (A), D2.2 (A), J1.1 (Pin_1), J2.1 (Pin_1)
- net IO17: now reaches U1.10 (IO17)
- net IO17: now also R8.1
- net IO18: now reaches U1.11 (IO18)
- net IO18: now also R9.1
- net IO15: now reaches U1.8 (IO15)
- net IO15: now also SW1.1
- net IO16: now reaches U1.9 (IO16)
- net IO16: now also SW2.1
- net IO4 renamed J1x
- net J1x: now also J1.3 (Pin_3); no longer SW1.1
- net IO5 renamed J1y
- net J1y: now also J1.4 (Pin_4); no longer SW2.1
- net IO6 renamed J2x
- net J2x: now also J2.3 (Pin_3)
- net IO7 renamed J2y
- net J2y: now also J2.4 (Pin_4)
- new net: R10.1, R11.2
- new net: D3.1 (K), R10.2
- new net: D2.1 (K), R9.2
- new net: D1.1 (K), R8.2
- no-connect marks 33 -> 29

Commit message: sep 18
Parts:
- added H3, H4, H5: MountingHole, MountingHole:MountingHole_2.5mm, symbol Mechanical:MountingHole
Connections:
- net IO13: now reaches J2.5 (Pin_5)
- net IO13: now also U1.21 (IO13)
- net IO12: now reaches J1.5 (Pin_5)
- net IO12: now also U1.20 (IO12)
- no-connect marks 29 -> 27
Other:
- moved on the sheet: H1, H2

Commit message: readme more
Connections:
- net +3.3V: no longer D3.2 (A), R1.1, R2.1, R5.2, USBC1.A1B12 (GND), USBC1.B1A12 (GND)
- net +5V: no longer C14.2, C15.1, R3.2, U2.1 (VINA), U2.10 (VIN), U2.11 (VIN), U2.12 (EN)
- net +5VA: now also C14.2, C15.1, R3.2, U2.1 (VINA), U2.10 (VIN), U2.11 (VIN), U2.12 (EN)
- new net GND1: D3.2 (A), R1.1, R2.1, R5.2, USBC1.A1B12 (GND), USBC1.B1A12 (GND)
