File: kicad/drone/lux.kicad_pcb (KiCad board)
At the start: 4 copper layers, 94 x 28 mm, 50 parts, among them M1 Motor_DC, M2 Motor_DC, M3 Motor_DC, M4 Motor_DC, T1 trace, U1 ESP32-S3-WROOM-1U-N16R8, U2 TPS63020DSJR

Commit message: done
Parts:
- moved C9 1.50 mm to (1163.5, 1042.0)
- moved M1 1.00 mm to (1164.5, 1037.0)
- moved M3 0.45 mm to (1231.0, 1058.0)
Routing:
- net /M1A: track 16.9 -> 18.5 mm
- net /M1B: track 15.6 -> 16.2 mm
Changed lines of the file:
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@@
 	(footprint "Connector_JST:JST_PH_B2B-PH-K_1x02_P2.00mm_Vertical"
 		(layer "F.Cu")
-		(at 1231 1058.45)
+		(at 1231 1058)
 		(descr "JST PH series connector, B2B-PH-K (http://www.jst-mfg.com/product/pdf/eng/ePH.pdf)")
 		(tags "connector JST PH vertical")
@@
 	(footprint "Capacitor_SMD:C_1206_3216Metric"
 		(layer "F.Cu")
-		(at 1163.5 1040.5)
+		(at 1163.5 1042)
 		(descr "Capacitor SMD 1206 (3216 Metric), square (rectangular) end terminal, IPC-7351 nominal, (Body size source: IPC-SM-782 page 76, https://www.pcb-3d.com/wordpress/wp-content/uploads/ipc-sm-782a_amendment_1_and_2.pdf)")
 		(tags "capacitor")
@@
 	(footprint "Connector_JST:JST_PH_B2B-PH-K_1x02_P2.00mm_Vertical"
 		(layer "F.Cu")
-		(at 1164.5 1036)
+		(at 1164.5 1037)
 		(descr "JST PH series connector, B2B-PH-K (http://www.jst-mfg.com/product/pdf/eng/ePH.pdf)")
 		(tags "connector JST PH vertical")
@@
 	)
 	(segment
+		(start 1162.025 1040.5)
+		(end 1162.025 1041.1)
+		(width 0.6)
+		(layer "F.Cu")
+		(net "/M1A")
+	)
+	(segment
 		(start 1156.37 1042.32)
 		(end 1156.37 1040.32)
@@
 	)
 	(segment
+		(start 1164.5 1036)
+		(end 1164.5 1037)
+		(width 1)
+		(layer "In1.Cu")
+		(net "/M1A")
+	)
+	(segment
 		(start 1163 1036)
 		(end 1162.025 1036.975)
@@
 	)
 	(segment
+		(start 1164.975 1040.5)
+		(end 1164.975 1041.1)
+		(width 0.6)
+		(layer "F.Cu")
+		(net "/M1B")
+	)
+	(segment
